File: hallpico.kicad_sch (KiCad schematic)
At the start: 20 parts, among them J1 BOOT Jump Wire, SW1 SW_SPST, SW2 SW_SPST, U1 RP2040 MiniPico V1.1, U2 GH39FKSW, U3 GH39FKSW, U4 GH39FKSW, U5 GH39FKSW

Commit message: fix: pro micro not mini pico
Parts:
- U1: value RP2040 MiniPico V1.1 -> RP2040 Pro Micro; footprint Library:RP2040_MiniPico_V1.1 -> Library:RP2040_ProMicro; symbol Library:RP2040_MiniPico_V1.1 -> Library:RP2040_ProMicro
Changed lines of the file:
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@@
 	)
 	(symbol
-		(lib_id "Library:RP2040_MiniPico_V1.1")
+		(lib_id "Library:RP2040_ProMicro")
 		(at 104.14 63.5 0)
 		(unit 1)
@@
 			)
 		)
-		(property "Value" "RP2040 MiniPico V1.1"
+		(property "Value" "RP2040 Pro Micro"
 			(at 114.3 60.96 0)
 			(effects
@@
 			)
 		)
-		(property "Footprint" "Library:RP2040_MiniPico_V1.1"
+		(property "Footprint" "Library:RP2040_ProMicro"
 			(at 114.046 59.436 0)
 			(effects
@@
 			)
 		)
-		(property "Description" "RP2040 ProMicro (MiniPico) Board from nologotech"
+		(property "Description" "RP2040 Pro Micro Board from nologotech"
 			(at 107.696 54.61 0)
 			(effects
