File: hallpico.kicad_pcb (KiCad board)
At the start: 2 copper layers, 61 x 58.4 mm, 20 parts, among them J1 BOOT Jump Wire, SW1 SW_SPST, SW2 SW_SPST, U1 RP2040 MiniPico V1.1, U2 GH39FKSW, U3 GH39FKSW, U4 GH39FKSW, U5 GH39FKSW

Commit message: fix: update board with naming fix
Parts:
- H1: moved to F.Cu
- U1: value RP2040 MiniPico V1.1 -> RP2040 Pro Micro; footprint Library:RP2040_MiniPico_V1.1 -> Library:RP2040_ProMicro
- turned H1 to 0 degrees

Commit message: fix: cleanup
Parts:
- moved U1 37.2 mm to (72.3, 46.9), turned to 180 degrees
Routing:
- net +3V3: track 122.5 -> 68.8 mm
- net LED_DIN: track 64.6 -> 19.3 mm
- net RST: track 60.2 -> 16.8 mm
- net ADC2: track 50.2 -> 29.1 mm, vias 2 -> 1
- net ADC3: track 52.4 -> 31.6 mm, vias 2 -> 1
- net ADC1: track 51.7 -> 32.6 mm
- net ADC0: track 30.1 -> 14.5 mm, vias 1 -> 0
- net +5V: track 125.7 -> 115.2 mm, vias 0 -> 2
- net GND: vias 0 -> 22
